File: WSPR_beacon/Schematics/WSPR_WilHam_Repeater/WSPR_WilHam_Repeater.kicad_sch (KiCad schematic)
At the start: 38 parts, among them J1 USB_C_Receptacle, J2 1PPS, J3 Conn_Coaxial, Q1 AO3401A, Q2 BS170, SW1 SW_SPDT_321, T1 bifilar 10T, U1 ATGM336H, U2 LTC4054ES5, U3 TLV1117-33, U4 ESP32-S3-WROOM-1, U5 Si5351A-A-GT, X1 IQXO-70

Commit message: Schematic Done
Parts:
- added C15, C16, C17, C18, C19: 100nF, Capacitor_SMD:C_0805_2012Metric, symbol Device:C_Small
- added D2, D3: LED_KRGB, symbol Device:LED_KRGB
- added H1, H2, H3, H4: MountingHole, MountingHole:MountingHole_2.2mm_M2, symbol Mechanical:MountingHole
- added J4: OledDisplay, Connector_PinHeader_2.54mm:PinHeader_1x04_P2.54mm_Vertical, symbol Connector_Generic:Conn_01x04
- added J5: Conn_01x04, symbol Connector_Generic:Conn_01x04
- added J6: Conn_01x03, symbol Connector_Generic:Conn_01x03
- added JP2: JOpen, Jumper:SolderJumper-2_P1.3mm_Open_TrianglePad1.0x1.5mm, symbol Jumper:Jumper_2_Open
- added JP3: JClosed, Jumper:SolderJumper-2_P1.3mm_Bridged_Pad1.0x1.5mm, symbol Jumper:Jumper_2_Bridged
- added JP4: Jumper_2_Open, Jumper:SolderJumper-2_P1.3mm_Open_TrianglePad1.0x1.5mm, symbol Jumper:Jumper_2_Open
- added JP5: Jumper_2_Bridged, Jumper:SolderJumper-2_P1.3mm_Bridged_Pad1.0x1.5mm, symbol Jumper:Jumper_2_Bridged
- added R4, R5: R_Small, symbol Device:R_Small
- added R6: 1M, Resistor_SMD:R_0805_2012Metric, symbol Device:R_Small
- added RN2: R_Pack04, symbol Device:R_Pack04
- added SW2: SW_Push, symbol Switch:SW_Push
- added SW3: Rotary_Encoder_Switch, cafebabe:EC11L1524E03_Rotary_Encoder, symbol Device:Rotary_Encoder_Switch
- C14: value 10uF -> 22uF
Connections:
- net Reset is gone; now on net GPS_Reset: U1.9 (nRESET)
- net CLK2: now also U4.7 (IO7)
- net D+: now also U4.14 (IO20)
- net D-: now also U4.13 (IO19)
- net GPS_En: now also U4.39 (IO1), J6.1 (Pin_1)
- net GPS_RX: now also U4.15 (IO3), J6.3 (Pin_3)
- net GPS_TX: now also U4.38 (IO2), J6.2 (Pin_2)
- net RX: now also J5.3 (Pin_3)
- net SCL: now also U4.5 (IO5), J4.2 (Pin_2), RN2.2 (R2.1)
- net SDA: now also U4.6 (IO6), J4.1 (Pin_1), RN2.1 (R1.1)
- net TX: now also J5.2 (Pin_2)
- net VCC: now also C15.1, C17.1, J5.1 (Pin_1), JP2.1 (A), JP5.2 (B), R6.2, RN2.7 (R2.2), RN2.8 (R1.2)
- net VSS: now also C15.2, C16.2, C17.2, C18.2, C19.1, J5.4 (Pin_4), JP3.1 (A), JP4.1 (A), R4.1, R5.1, SW2.1, SW3.C, SW3.S1
- net RotaryS: now reaches U4.18 (IO10)
- net RotaryS: now also SW3.S2
- net RotaryA: now reaches U4.19 (IO11)
- net RotaryA: now also C18.1, SW3.B
- net RotaryB: now reaches U4.20 (IO12)
- net RotaryB: now also C19.2, SW3.A
- net R1: now reaches U4.28 (IO35)
- net R1: now also D2.2 (RA)
- net G1: now reaches U4.29 (IO36)
- net G1: now also D2.3 (GA)
- net at U4.3 (EN): now also C16.1, R6.1, SW2.2
- net B1: now reaches U4.30 (IO37)
- net B1: now also D2.4 (BA)
- net R2: now reaches U4.31 (IO38)
- net R2: now also D3.2 (RA)
- net G2: now reaches U4.32 (IO39)
- net G2: now also D3.3 (GA)
- net B2: now reaches U4.33 (IO40)
- net B2: now also D3.4 (BA)
- net GPS_Reset: now reaches U4.4 (IO4)
- new net: J4.3 (Pin_3), JP4.2 (B), JP5.1 (A)
- new net: D2.1 (K), R4.2
- new net: J4.4 (Pin_4), JP2.2 (B), JP3.2 (B)
- new net: D3.1 (K), R5.2
- no-connect marks 19 -> 23
Other:
- moved on the sheet: AE1, BT1, C10, C11, C12, C13, C14, C2, J2, J3, L1, Q2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
